Commit message: Rename finger_left to left_finger

File: rg6_gripper_description/urdf/rg6_gripper.urdf.xacro (robot description, xacro)
@@ -55,5 +55,5 @@
         </xacro:macro>
         <!-- FINGER LEFT -->
-        <joint name="${prefix}_finger_left_joint" type="revolute">
+        <joint name="${prefix}_left_finger_joint" type="revolute">
             <limit lower="-0.85" upper="0.47" effort="1.0" velocity="0.6"/>
             <axis xyz="0 0 1"/>
@@ -69,5 +69,5 @@
                 <motorTorqueConstant>1</motorTorqueConstant>
             </actuator>
-            <joint name="${prefix}_finger_left_joint" >
+            <joint name="${prefix}_left_finger_joint" >
                 <hardwareInterface>hardware_interface/PositionJointInterface</hardwareInterface>
             </joint>
@@ -103,5 +103,5 @@
         </gazebo>
          <!-- THUMB LEFT -->
-        <joint name="${prefix}_thumb_left_joint" type="revolute">
+        <joint name="${prefix}_left_thumb_joint" type="revolute">
             <limit lower="-2.0" upper="2.0" effort="1.0" velocity="0.0125"/>
             <axis xyz="0 0 1"/>
@@ -110,8 +110,8 @@
             <child link="${prefix}_left_thumb" />
             <dynamics friction="100" damping="100" />
-            <mimic joint="${prefix}_finger_left_joint" multiplier="-1.0" offset="0"/>
-        </joint>
-        <xacro:mimic_joint_plugin_gazebo parent_joint="${prefix}_finger_left_joint"
-                                         mimic_joint="${prefix}_thumb_left_joint" has_pid="false" multiplier="-1.0" max_effort="10.0" />
+            <mimic joint="${prefix}_left_finger_joint" multiplier="-1.0" offset="0"/>
+        </joint>
+        <xacro:mimic_joint_plugin_gazebo parent_joint="${prefix}_left_finger_joint"
+                                         mimic_joint="${prefix}_left_thumb_joint" has_pid="false" multiplier="-1.0" max_effort="10.0" />
         <link name="${prefix}_left_thumb">
             <inertial>
@@ -140,5 +140,5 @@
         </link>
         <!-- FINGER RIGHT -->
-        <joint name="${prefix}_finger_right_joint" type="revolute">
+        <joint name="${prefix}_right_finger_joint" type="revolute">
             <limit lower="-0.85" upper="0.47" effort="1.0" velocity="0.6"/>
             <axis xyz="0 0 1"/>
@@ -147,8 +147,8 @@
             <child link="${prefix}_right_finger" />
             <dynamics damping="0" friction="0"/>
-            <mimic joint="${prefix}_finger_left_joint" multiplier="-1.0" offset="0"/>
-        </joint>
-        <xacro:mimic_joint_plugin_gazebo parent_joint="${prefix}_finger_left_joint"
-                                         mimic_joint="${prefix}_finger_right_joint" has_pid="false" multiplier="-1.0" max_effort="10.0" />
+            <mimic joint="${prefix}_left_finger_joint" multiplier="-1.0" offset="0"/>
+        </joint>
+        <xacro:mimic_joint_plugin_gazebo parent_joint="${prefix}_left_finger_joint"
+                                         mimic_joint="${prefix}_right_finger_joint" has_pid="false" multiplier="-1.0" max_effort="10.0" />
         <link name="${prefix}_right_finger">
             <inertial>
@@ -181,5 +181,5 @@
         </gazebo>
          <!-- THUMB RIGHT -->
-        <joint name="${prefix}_thumb_right_joint" type="revolute">
+        <joint name="${prefix}_right_thumb_joint" type="revolute">
             <limit lower="-2.0" upper="2.0" effort="1.0" velocity="0.0125"/>
             <axis xyz="0 0 1"/>
@@ -188,8 +188,8 @@
             <child link="${prefix}_right_thumb" />
             <dynamics friction="100" damping="100" />
-            <mimic joint="${prefix}_finger_right_joint" multiplier="-1.0" offset="0"/>
-        </joint>
-        <xacro:mimic_joint_plugin_gazebo parent_joint="${prefix}_finger_left_joint"
-                                         mimic_joint="${prefix}_thumb_right_joint" has_pid="false" multiplier="1.0" max_effort="10.0" />
+            <mimic joint="${prefix}_right_finger_joint" multiplier="-1.0" offset="0"/>
+        </joint>
+        <xacro:mimic_joint_plugin_gazebo parent_joint="${prefix}_left_finger_joint"
+                                         mimic_joint="${prefix}_right_thumb_joint" has_pid="false" multiplier="1.0" max_effort="10.0" />
         <link name="${prefix}_right_thumb">
             <inertial>
